File: UI.sch (KiCad schematic (older format))
At the start: 7 parts, among them SW1 Rotary_Encoder_Switch, SW2 PTT, SW3 Left, SW4 Right

Commit message: Almost final PCB
Parts:
- SW2: footprint Button_Switch_THT:SW_PUSH_6mm -> uSDX:Limit
Changed lines of the file:
@@
 F 0 "SW2" H 4500 3585 50  0000 C CNN
 F 1 "PTT" H 4500 3494 50  0000 C CNN
-F 2 "Button_Switch_THT:SW_PUSH_6mm" H 4500 3500 50  0001 C CNN
+F 2 "uSDX:Limit" H 4500 3500 50  0001 C CNN
 F 3 "~" H 4500 3500 50  0001 C CNN
 	1    4500 3300
