File: _autosave-Audio.sch (KiCad schematic (older format))
At the start: 24 parts, among them J5 Mic, J6 Headphones, U8 LM386

Commit message: Almost final PCB
Parts:
- gave numbers to parts that had none: 2
Changed lines of the file:
@@
 P 4200 2500
 AR Path="/60EE260F" Ref="L?"  Part="1"
-AR Path="/610D2463/60EE260F" Ref="L?"  Part="1"
-F 0 "L?" V 4390 2500 50  0000 C CNN
+AR Path="/610D2463/60EE260F" Ref="L5"  Part="1"
+F 0 "L5" V 4390 2500 50  0000 C CNN
 F 1 "100uH" V 4299 2500 50  0000 C CNN
 F 2 "Inductor_SMD:L_0805_2012Metric_Pad1.15x1.40mm_HandSolder" H 4200 2500 50  0001 C CNN
@@
 $EndComp
 $Comp
-L power:VCC #PWR?
+L power:VCC #PWR053
 U 1 1 60EE4AA8
 P 4500 2350
-F 0 "#PWR?" H 4500 2200 50  0001 C CNN
+F 0 "#PWR053" H 4500 2200 50  0001 C CNN
 F 1 "VCC" H 4515 2523 50  0000 C CNN
 F 2 "" H 4500 2350 50  0001 C CNN
@@
 P 3900 2800
 AR Path="/60EF36F1" Ref="C?"  Part="1"
-AR Path="/610D2463/60EF36F1" Ref="C?"  Part="1"
-F 0 "C?" H 3785 2754 50  0000 R CNN
+AR Path="/610D2463/60EF36F1" Ref="C12"  Part="1"
+F 0 "C12" H 3785 2754 50  0000 R CNN
 F 1 "100n" H 3785 2845 50  0000 R CNN
 F 2 "Capacitor_SMD:C_0805_2012Metric_Pad1.18x1.45mm_HandSolder" H 3938 2650 50  0001 C CNN
@@
 P 3900 3000
 AR Path="/60F00371" Ref="#PWR?"  Part="1"
-AR Path="/610D2463/60F00371" Ref="#PWR?"  Part="1"
-F 0 "#PWR?" H 3900 2750 50  0001 C CNN
+AR Path="/610D2463/60F00371" Ref="#PWR018"  Part="1"
+F 0 "#PWR018" H 3900 2750 50  0001 C CNN
 F 1 "GND" H 3905 2827 50  0000 C CNN
 F 2 "" H 3900 3000 50  0001 C CNN
