File: uSDX.kicad_pcb (KiCad board)
At the start: 2 copper layers, 123 parts, among them J1 Jack-DC, J2 GPS_CONN, J3 ICSP, J4 SMA, J5 Mic, J6 Headphones, Q1 2N7002, Q2 IRLML2060, Q3 2N7002, Q4 2N7002, SW1 Rotary_Encoder_Switch, SW2 PTT, SW3 Left, SW4 Right, T1 SWR, U1 L7805, U2 LD1117S33TR_SOT223, U3 ATmega328PB-AU, U4 LM4562, U5 74AHCT1G00, U6 SN74CBT3253, U7 Filter, U8 LM386, U9 Si5351A-B-GT, X1 FT3HNBPK27.0-T1, Y1 20MHz

Commit message: Work on PCB
Parts:
- added Q5: IRLML2060, Package_TO_SOT_SMD:SOT-23, F.Cu at (43.2, -44.5)
- added Q6: IRLML2060, Package_TO_SOT_SMD:SOT-23, F.Cu at (43.2, -36.8)
- added REF**: MountingHole_3.2mm_M3_DIN965_Pad, MountingHole:MountingHole_3.2mm_M3_DIN965_Pad, F.Cu at (70.0, -100.0)
- added REF**: MountingHole_3.2mm_M3_DIN965_Pad, MountingHole:MountingHole_3.2mm_M3_DIN965_Pad, F.Cu at (70.0, -10.0)
- added REF**: MountingHole_3.2mm_M3_DIN965_Pad, MountingHole:MountingHole_3.2mm_M3_DIN965_Pad, F.Cu at (160.0, -10.0)
- added REF**: MountingHole_3.2mm_M3_DIN965_Pad, MountingHole:MountingHole_3.2mm_M3_DIN965_Pad, F.Cu at (160.0, -100.0)
- moved J2 248.7 mm to (0.64, -84.5)
- moved U3 243.9 mm to (109.2, -81.9)
- moved Y1 243.7 mm to (101.6, -80.0)
- moved C11 243.3 mm to (121.9, -81.9)
- moved C10 241.7 mm to (101.0, -83.2)
- moved C8 240.5 mm to (101.0, -85.1)
- moved L3 237.5 mm to (123.8, -81.9)
- moved J3 233.0 mm to (20.3, -61.0)
- moved R1 227.4 mm to (109.9, -90.8), turned to 270 degrees
- moved JP1 218.8 mm to (108.6, -97.2)
- moved JP2 218.5 mm to (113.0, -97.2)
- moved C12 217.3 mm to (108.0, -90.8), turned to 270 degrees
- moved C9 214.3 mm to (116.2, -81.9), turned to 270 degrees
- moved R19 212.5 mm to (129.4, -41.3), turned to 0 degrees
- moved MK1 211.6 mm to (141.6, -38.7), turned to 0 degrees
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Connections:
- J5 pad R: (no net) -> PB5
- J5 pad RN: (no net) -> Net-(J5-PadRN)
- J5 pad S: PB4 -> GND
- J5 pad T: PB5 -> PB4
- J6 pad R: (no net) -> Net-(C34-Pad2)
- J6 pad RN: (no net) -> Net-(J6-PadRN)
- J6 pad S: Net-(C34-Pad2) -> GND
- LS1 pad 2: Net-(J6-PadSN) -> Net-(J6-PadRN)
- MK1 pad 2: Net-(J5-PadSN) -> Net-(J5-PadTN)
Routing:
- net GND: track 7.81 -> 240.7 mm
- net +3V3: track 0.00 -> 47.8 mm, vias 0 -> 3
- net +12V: track 0.00 -> 40.0 mm
- net /RF/RF: track 0.00 -> 35.1 mm
- net Net-(D3-Pad1): track 0.00 -> 30.6 mm
- net Net-(C34-Pad2): track 0.00 -> 30.5 mm
- net /SWR/RF_OUT: track 0.00 -> 28.2 mm
- net /PLL/CLK_I: track 0.00 -> 18.0 mm, vias 0 -> 2
- net Net-(C16-Pad2): track 0.00 -> 16.6 mm
- net Net-(C34-Pad1): track 0.00 -> 15.2 mm
- net Net-(J6-PadRN): track 0.00 -> 14.9 mm
- net Net-(C30-Pad1): track 5.31 -> 16.4 mm
- net VCC: track 7.45 -> 17.1 mm
- net Net-(C20-Pad1): track 0.00 -> 9.24 mm
- net /PLL/CLK_Q: track 0.00 -> 8.39 mm
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Other:
- board outline added: 100 x 100 mm

Commit message: Almost final PCB
Parts:
- added L5: 100uH, Inductor_SMD:L_0805_2012Metric_Pad1.15x1.40mm_HandSolder, F.Cu at (130.2, -42.5)
- JP1, JP2: moved to B.Cu
- SW2: footprint Button_Switch_THT:SW_PUSH_6mm -> uSDX:Limit
- moved J2 126.4 mm to (127.0, -88.9)
- moved C43 111.8 mm to (108.1, -66.7), turned to 180 degrees
- moved C44 107.8 mm to (111.3, -62.9), turned to 270 degrees
- moved X1 106.6 mm to (108.1, -62.9), turned to 0 degrees
- moved R25 105.6 mm to (104.9, -62.9), turned to 270 degrees
- moved R26 105.1 mm to (103.0, -62.9), turned to 90 degrees
- moved C45 101.2 mm to (113.8, -57.1), turned to 90 degrees
- moved R27 100.1 mm to (106.8, -58.4), turned to 90 degrees
- moved U9 99.8 mm to (110.6, -57.1), turned to 270 degrees
- moved Q3 99.1 mm to (103.6, -58.4), turned to 180 degrees
- moved R29 98.3 mm to (100.5, -58.4), turned to 90 degrees
- moved C32 94.3 mm to (120.8, -48.3), turned to 270 degrees
- moved R28 94.0 mm to (106.8, -54.0), turned to 90 degrees
- moved R15 93.1 mm to (118.9, -48.3), turned to 270 degrees
- moved Q4 92.9 mm to (103.6, -54.0), turned to 180 degrees
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Connections:
- C12 pad 1: GND -> Net-(C12-Pad1)
- C12 pad 2: RST -> GND
- J2 pad 1: PPS -> PD2
- R19 pad 1: +5VA -> Net-(C12-Pad1)
- SW3 pad 2: PD0 -> PE0
- SW4 pad 2: PD1 -> PD5
- U3 pad 3: Net-(U3-Pad3) -> PE0
- U3 pad 30: PD0 -> RX
- U3 pad 31: PD1 -> TX
- U3 pad 9: Net-(U3-Pad9) -> PD5
Routing:
- net GND: track 240.7 -> 440.6 mm, vias 0 -> 14
- net VCC: track 17.1 -> 197.2 mm, vias 0 -> 10
- net +12V: track 40.0 -> 199.2 mm
- net PD5: track 0.00 -> 124.4 mm
- net PD4: track 0.00 -> 107.1 mm, vias 0 -> 2
- net PD7: track 0.00 -> 97.7 mm, vias 0 -> 2
- net PB5: track 0.00 -> 92.0 mm, vias 0 -> 3
- net +3V3: track 47.8 -> 139.8 mm, vias 3 -> 9
- net PE0: track 0.00 -> 90.5 mm, vias 0 -> 2
- net PD6: track 0.00 -> 90.4 mm, vias 0 -> 2
- net PB4: track 0.00 -> 80.6 mm, vias 0 -> 1
- net AREF: track 2.45 -> 73.7 mm, vias 0 -> 4
- net ADC2: track 0.00 -> 69.2 mm, vias 0 -> 4
- net SCL: track 2.59 -> 64.9 mm, vias 0 -> 4
- net SDA: track 2.59 -> 58.1 mm, vias 0 -> 4
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- added copper zone on B.Cu, net GND
- added copper zone on F.Cu, net GND

Commit message: Final
Parts:
- added ADC0: TestPoint_Pad_D1.0mm, TestPoint:TestPoint_Pad_D1.0mm, F.Cu at (122.6, -48.9)
- added ADC1: TestPoint_Pad_D1.0mm, TestPoint:TestPoint_Pad_D1.0mm, F.Cu at (123.2, -54.6)
Routing:
- net ADC1: track 58.7 -> 62.5 mm
- net ADC0: track 45.5 -> 47.4 mm
- net PB4: track 80.6 -> 81.2 mm
Other:
- board text added: "2021"
- board text added: "GPS"
- board text added: "Headphones"
- board text added: "ICSP"
- board text added: "Microphone"
- board text added: "Speaker"
- board text added: "by knowak.xyz & Jelcz Industries"
- board text added: "uSDX"
