File: filter/filter.sch (KiCad schematic (older format))
At the start: 10 parts, among them J101 TRX, J102 TRX

Commit message: PCB in progress, filter screwed up
Parts:
- removed J101, J102: TRX, Connector_PinHeader_2.54mm:PinHeader_1x04_P2.54mm_Vertical, symbol Connector:Conn_01x04_Male
- added R1: 10.875, symbol Device:R
- added R2: 50, symbol Device:R
- added V1: VSIN, symbol Simulation_SPICE:VSIN
- C105: value 620p -> 1600p
- C106: value 470p -> 1600p
- L101: value 675n -> 900n
- L102: value 243n -> 413n
Connections:
- wire segments 25 -> 31
Changed lines of the file:
@@
 P 5250 3500
 F 0 "L101" V 5440 3500 50  0000 C CNN
-F 1 "675n" V 5349 3500 50  0000 C CNN
+F 1 "900n" V 5349 3500 50  0000 C CNN
 F 2 "Inductor_THT:L_Toroid_Horizontal_D9.5mm_P15.00mm_Diameter10-5mm_Amidon-T37" H 5250 3500 50  0001 C CNN
 F 3 "~" H 5250 3500 50  0001 C CNN
@@
 P 6000 3750
 F 0 "C105" H 5885 3704 50  0000 R CNN
-F 1 "620p" H 5885 3795 50  0000 R CNN
+F 1 "1600p" H 5885 3795 50  0000 R CNN
 F 2 "Capacitor_SMD:C_0805_2012Metric_Pad1.18x1.45mm_HandSolder" H 6038 3600 50  0001 C CNN
 F 3 "~" H 6000 3750 50  0001 C CNN
@@
 P 6250 3500
 F 0 "L102" V 6440 3500 50  0000 C CNN
-F 1 "243n" V 6349 3500 50  0000 C CNN
+F 1 "413n" V 6349 3500 50  0000 C CNN
 F 2 "Inductor_THT:L_Toroid_Horizontal_D9.5mm_P15.00mm_Diameter10-5mm_Amidon-T37" H 6250 3500 50  0001 C CNN
 F 3 "~" H 6250 3500 50  0001 C CNN
@@
 P 6500 3750
 F 0 "C106" H 6385 3704 50  0000 R CNN
-F 1 "470p" H 6385 3795 50  0000 R CNN
+F 1 "1600p" H 6385 3795 50  0000 R CNN
 F 2 "Capacitor_SMD:C_0805_2012Metric_Pad1.18x1.45mm_HandSolder" H 6538 3600 50  0001 C CNN
 F 3 "~" H 6500 3750 50  0001 C CNN
@@
 Wire Wire Line
 	7000 3500 6500 3500
-Wire Wire Line
-	5000 3500 4500 3500
-Connection ~ 5000 3500
 $Comp
 L power:GND #PWR0101
@@
 Wire Wire Line
 	4650 3800 4500 3800
-$Comp
-L power:GND #PWR0102
-U 1 1 61019A2B
-P 6850 3900
-F 0 "#PWR0102" H 6850 3650 50  0001 C CNN
-F 1 "GND" H 6855 3727 50  0000 C CNN
-F 2 "" H 6850 3900 50  0001 C CNN
-F 3 "" H 6850 3900 50  0001 C CNN
-	1    6850 3900
-	1    0    0    -1
-$EndComp
-Wire Wire Line
-	6850 3900 6850 3800
-Wire Wire Line
-	6850 3800 7000 3800
-$Comp
-L Connector:Conn_01x04_Male J101
-U 1 1 6101E0B1
-P 4300 3600
-F 0 "J101" H 4408 3881 50  0000 C CNN
-F 1 "TRX" H 4408 3790 50  0000 C CNN
-F 2 "Connector_PinHeader_2.54mm:PinHeader_1x04_P2.54mm_Vertical" H 4300 3600 50  0001 C CNN
-F 3 "~" H 4300 3600 50  0001 C CNN
-	1    4300 3600
-	1    0    0    -1
-$EndComp
-$Comp
-L Connector:Conn_01x04_Male J102
-U 1 1 61024C76
-P 7200 3600
-F 0 "J102" H 7172 3574 50  0000 R CNN
-F 1 "TRX" H 7172 3483 50  0000 R CNN
-F 2 "Connector_PinHeader_2.54mm:PinHeader_1x04_P2.54mm_Vertical" H 7200 3600 50  0001 C CNN
-F 3 "~" H 7200 3600 50  0001 C CNN
-	1    7200 3600
-	-1   0    0    -1
-$EndComp
+Wire Wire Line
+	3800 4200 4500 4200
+Wire Wire Line
+	4500 4200 4500 3800
+$Comp
+L Simulation_SPICE:VSIN V1
+U 1 1 60FD3107
+P 3800 3750
+F 0 "V1" H 3930 3841 50  0000 L CNN
+F 1 "VSIN" H 3930 3750 50  0000 L CNN
+F 2 "" H 3800 3750 50  0001 C CNN
+F 3 "~" H 3800 3750 50  0001 C CNN
+F 4 "Y" H 3800 3750 50  0001 L CNN "Spice_Netlist_Enabled"
+F 5 "V" H 3800 3750 50  0001 L CNN "Spice_Primitive"
+F 6 "ac 1" H 3930 3659 50  0000 L CNN "Spice_Model"
+	1    3800 3750
+	1    0    0    -1
+$EndComp
+Wire Wire Line
+	3800 3950 3800 4200
+$Comp
+L Device:R R2
+U 1 1 60FD8214
+P 7000 3800
+F 0 "R2" H 7070 3846 50  0000 L CNN
+F 1 "50" H 7070 3755 50  0000 L CNN
+F 2 "" V 6930 3800 50  0001 C CNN
+F 3 "~" H 7000 3800 50  0001 C CNN
+	1    7000 3800
+	1    0    0    -1
+$EndComp
+Wire Wire Line
+	7000 3650 7000 3500
+$Comp
+L power:GND #PWR01
+U 1 1 60FD8CF5
+P 7000 4050
+F 0 "#PWR01" H 7000 3800 50  0001 C CNN
+F 1 "GND" H 7005 3877 50  0000 C CNN
+F 2 "" H 7000 4050 50  0001 C CNN
+F 3 "" H 7000 4050 50  0001 C CNN
+	1    7000 4050
+	1    0    0    -1
+$EndComp
+Wire Wire Line
+	7000 4050 7000 3950
+$Comp
+L Device:R R1
+U 1 1 60FDA494
+P 4450 3450
+F 0 "R1" V 4243 3450 50  0000 C CNN
+F 1 "10.875" V 4334 3450 50  0000 C CNN
+F 2 "" V 4380 3450 50  0001 C CNN
+F 3 "~" H 4450 3450 50  0001 C CNN
+	1    4450 3450
+	0    1    1    0
+$EndComp
+Wire Wire Line
+	5000 3500 4600 3500
+Wire Wire Line
+	4600 3500 4600 3450
+Connection ~ 5000 3500
+Wire Wire Line
+	4300 3450 3800 3450
+Wire Wire Line
+	3800 3450 3800 3550
 $EndSCHEMATC

Commit message: Reverted filter
Parts:
- removed R1: 10.875, symbol Device:R
- removed R2: 50, symbol Device:R
- removed V1: VSIN, symbol Simulation_SPICE:VSIN
- added J101, J102: TRX, Connector_PinHeader_2.54mm:PinHeader_1x04_P2.54mm_Vertical, symbol Connector:Conn_01x04_Male
- C105: value 1600p -> 620p
- C106: value 1600p -> 470p
- L101: value 900n -> 675n
- L102: value 413n -> 243n
Connections:
- wire segments 31 -> 25
Changed lines of the file:
@@
 P 5250 3500
 F 0 "L101" V 5440 3500 50  0000 C CNN
-F 1 "900n" V 5349 3500 50  0000 C CNN
+F 1 "675n" V 5349 3500 50  0000 C CNN
 F 2 "Inductor_THT:L_Toroid_Horizontal_D9.5mm_P15.00mm_Diameter10-5mm_Amidon-T37" H 5250 3500 50  0001 C CNN
 F 3 "~" H 5250 3500 50  0001 C CNN
@@
 P 6000 3750
 F 0 "C105" H 5885 3704 50  0000 R CNN
-F 1 "1600p" H 5885 3795 50  0000 R CNN
+F 1 "620p" H 5885 3795 50  0000 R CNN
 F 2 "Capacitor_SMD:C_0805_2012Metric_Pad1.18x1.45mm_HandSolder" H 6038 3600 50  0001 C CNN
 F 3 "~" H 6000 3750 50  0001 C CNN
@@
 P 6250 3500
 F 0 "L102" V 6440 3500 50  0000 C CNN
-F 1 "413n" V 6349 3500 50  0000 C CNN
+F 1 "243n" V 6349 3500 50  0000 C CNN
 F 2 "Inductor_THT:L_Toroid_Horizontal_D9.5mm_P15.00mm_Diameter10-5mm_Amidon-T37" H 6250 3500 50  0001 C CNN
 F 3 "~" H 6250 3500 50  0001 C CNN
@@
 P 6500 3750
 F 0 "C106" H 6385 3704 50  0000 R CNN
-F 1 "1600p" H 6385 3795 50  0000 R CNN
+F 1 "470p" H 6385 3795 50  0000 R CNN
 F 2 "Capacitor_SMD:C_0805_2012Metric_Pad1.18x1.45mm_HandSolder" H 6538 3600 50  0001 C CNN
 F 3 "~" H 6500 3750 50  0001 C CNN
@@
 Wire Wire Line
 	7000 3500 6500 3500
+Wire Wire Line
+	5000 3500 4500 3500
+Connection ~ 5000 3500
 $Comp
 L power:GND #PWR0101
@@
 Wire Wire Line
 	4650 3800 4500 3800
-Wire Wire Line
-	3800 4200 4500 4200
-Wire Wire Line
-	4500 4200 4500 3800
-$Comp
-L Simulation_SPICE:VSIN V1
-U 1 1 60FD3107
-P 3800 3750
-F 0 "V1" H 3930 3841 50  0000 L CNN
-F 1 "VSIN" H 3930 3750 50  0000 L CNN
-F 2 "" H 3800 3750 50  0001 C CNN
-F 3 "~" H 3800 3750 50  0001 C CNN
-F 4 "Y" H 3800 3750 50  0001 L CNN "Spice_Netlist_Enabled"
-F 5 "V" H 3800 3750 50  0001 L CNN "Spice_Primitive"
-F 6 "ac 1" H 3930 3659 50  0000 L CNN "Spice_Model"
-	1    3800 3750
-	1    0    0    -1
-$EndComp
-Wire Wire Line
-	3800 3950 3800 4200
-$Comp
-L Device:R R2
-U 1 1 60FD8214
-P 7000 3800
-F 0 "R2" H 7070 3846 50  0000 L CNN
-F 1 "50" H 7070 3755 50  0000 L CNN
-F 2 "" V 6930 3800 50  0001 C CNN
-F 3 "~" H 7000 3800 50  0001 C CNN
-	1    7000 3800
-	1    0    0    -1
-$EndComp
-Wire Wire Line
-	7000 3650 7000 3500
-$Comp
-L power:GND #PWR01
-U 1 1 60FD8CF5
-P 7000 4050
-F 0 "#PWR01" H 7000 3800 50  0001 C CNN
-F 1 "GND" H 7005 3877 50  0000 C CNN
-F 2 "" H 7000 4050 50  0001 C CNN
-F 3 "" H 7000 4050 50  0001 C CNN
-	1    7000 4050
-	1    0    0    -1
-$EndComp
-Wire Wire Line
-	7000 4050 7000 3950
-$Comp
-L Device:R R1
-U 1 1 60FDA494
-P 4450 3450
-F 0 "R1" V 4243 3450 50  0000 C CNN
-F 1 "10.875" V 4334 3450 50  0000 C CNN
-F 2 "" V 4380 3450 50  0001 C CNN
-F 3 "~" H 4450 3450 50  0001 C CNN
-	1    4450 3450
-	0    1    1    0
-$EndComp
-Wire Wire Line
-	5000 3500 4600 3500
-Wire Wire Line
-	4600 3500 4600 3450
-Connection ~ 5000 3500
-Wire Wire Line
-	4300 3450 3800 3450
-Wire Wire Line
-	3800 3450 3800 3550
+$Comp
+L power:GND #PWR0102
+U 1 1 61019A2B
+P 6850 3900
+F 0 "#PWR0102" H 6850 3650 50  0001 C CNN
+F 1 "GND" H 6855 3727 50  0000 C CNN
+F 2 "" H 6850 3900 50  0001 C CNN
+F 3 "" H 6850 3900 50  0001 C CNN
+	1    6850 3900
+	1    0    0    -1
+$EndComp
+Wire Wire Line
+	6850 3900 6850 3800
+Wire Wire Line
+	6850 3800 7000 3800
+$Comp
+L Connector:Conn_01x04_Male J101
+U 1 1 6101E0B1
+P 4300 3600
+F 0 "J101" H 4408 3881 50  0000 C CNN
+F 1 "TRX" H 4408 3790 50  0000 C CNN
+F 2 "Connector_PinHeader_2.54mm:PinHeader_1x04_P2.54mm_Vertical" H 4300 3600 50  0001 C CNN
+F 3 "~" H 4300 3600 50  0001 C CNN
+	1    4300 3600
+	1    0    0    -1
+$EndComp
+$Comp
+L Connector:Conn_01x04_Male J102
+U 1 1 61024C76
+P 7200 3600
+F 0 "J102" H 7172 3574 50  0000 R CNN
+F 1 "TRX" H 7172 3483 50  0000 R CNN
+F 2 "Connector_PinHeader_2.54mm:PinHeader_1x04_P2.54mm_Vertical" H 7200 3600 50  0001 C CNN
+F 3 "~" H 7200 3600 50  0001 C CNN
+	1    7200 3600
+	-1   0    0    -1
+$EndComp
 $EndSCHEMATC
